File: hardware/teensy-integrated-revf/design/racecar-integrated-revf.kicad_pcb (KiCad board)
At the start: 4 copper layers, 150 x 155 mm, 193 parts, among them J1 POWER IN, J10 NET 3V3 UART SERVICE, J11 THROTTLE 0.5-4.5V, J12 BRAKE 0.5-4.5V, J13 PI 5 VIDEO 3V3 UART, J14 CAN, J2 SCREEN J10 ONLY, J3 TACH INPUT, J4 OIL 0.5-4.5V, J5 COOLANT NTC, J6 AEM 30-0300 ONLY, J8 GPS SMA FEMALE, J9 TO TEENSY VBAT/GND, Q1 MMBT3904, Q2 MMBT3904, Q3 AO4485 P-FET 40V, U1 Teensy 4.1 SOCKETED, U10 SN74LVC1G125, U11 LM2903B, U12 VO617A-3, U13 SN74LVC2G17, U14 LM4040 4.1, U15 TMUX1511, U16 TMUX1511, U17 ESP32-S3-WROOM-1-N8R2, U18 SN74LVC125A, U19 SN74LVC2G125, U2 TPS54560B 5V 5A BUCK, U20 SN74LVC1G125, U21 TCAN1042HGV-Q1, U3 TSR 1-2433, U4 SN74LVC1T45, U5 SN74LVC1T45, U6 TSR 1-2433, U7 ICM-42670-P, U8 NEO-M9N-00B, U9 TPS2553

Commit message: Rev F silkscreen: every connector named at the part; replacement F.Silkscreen layer
The silkscreen in the package already uploaded to PCBWay could not be built from
as-is. This ships a replacement F.Silkscreen gerber (pcbway/addon-silkscreen/).
verify_addon.py proves the other 12 layers and both drills geometry-identical to
the uploaded ZIP, and now exits 1 on any other difference.

Found and fixed:
- 12 field-terminal labels missing: complete_routes.py deleted silk text by
  STRING, so J5 had no name or pins and J3/J4/J11/J12 showed only "3 SIG".
- GPS SMA / PI 5 VIDEO UART 3V3 / RTC 3V NO CHARGE sat 28-44 mm from J8/J13/BT1
  (hard-coded from an older placement); J9, J10 and JP1 had no label at all.
- No reference designators are printed on this board, so names now carry them.
- Teensy socket orientation marks and a column-aligned crossed screen-harness
  table under J2; all text >= 0.9 mm high / 0.16 mm stroke.

New electrical/silk_legends.py is ONE table used by generate.py and addon_silk.py
(idempotent): names just above each terminal, left-aligned pin labels on their
pad rows, J13 "2 TX>PI 10" / "3 RX<PI 8", J9/J10/J14 pin labels, J8/JP1/JP2/BT1
names. It slides a crowded label along its column and raises rather than drop one.
verify.py: 1078 assertions (was 749), incl. every J/JP/BT part named within 6 mm,
harness digits checked against J2's nets, J13 TX/RX against Teensy pins 1/0.
DRC 0 (all severities) / unconnected 0 / ERC 0. render_gerber.py rasterises the
shipped .gbr itself for readback. Engineering ZIP re-exported.

3D: the SMA twin is now Molex 73251-2200 Horizontal, a right-angle THT jack with
the 901-143's pin pattern and frame. The old twin was the 132289 edge-mount
(wrong kind of part, rendered along the edge) - render only; the footprint and
Gerbers were always right. New render_stills.py rebuilds render/check/*.png and
the viewer preview; GLB/HTML/preview carry the new silk.

CAD only: unbuilt, unmeasured, not independently reviewed.
Other:
- board text added: "1"
- board text added: "1 +5V"
- board text added: "1 NTC"
- board text added: "1 VBAT"
- board text added: "2"
- board text added: "2 +5V"
- board text added: "2 3V3"
- board text added: "2 RET"
- board text added: "2 TX>PI 10"
- board text added: "25"
- board text added: "3"
- board text added: "3 RX<PI 8"
- board text added: "3 TX OUT"
- board text added: "4"
- board text added: "4 GND"
- board text added: "4 RX IN"
- board text added: "5 BOOT"
- board text added: "6 EN"
- board text added: "BT1 CR2032 RTC - NO CHARGER"
- board text added: "CANH"
- board text added: "CANL"
- board text added: "GND"
- board text added: "J1 10-20V IN"
- board text added: "J10"
- board text added: "J10 NET PROG 3V3"
- board text added: "J11 THROTTLE"
- board text added: "J12 BRAKE"
- board text added: "J13 PI 5 VIDEO 3V3"
- board text added: "J14 CAN"
- board text added: "J2"
- board text added: "J2 -> SCREEN J10: CROSSED"
- board text added: "J2 SCREEN"
- board text added: "J3 TACH"
- board text added: "J4 OIL"
- board text added: "J5 COOLANT"
- board text added: "J6 AEM AFR"
- board text added: "J8 GPS ANT"
- board text added: "J9 RTC LEAD"
- board text added: "JP1 TEENSY PWR"
- board text added: "JP2 CAN TERM: BUS END ONLY"
- board text added: "TEENSY"
- board text added: "THIS EDGE"
- board text added: "USB END"
- board text removed: "1 CANH"
- board text removed: "10-20V IN"
- board text removed: "2 CANL"
- board text removed: "3 GND"
- board text removed: "AEM AFR"
- board text removed: "BRAKE"
- board text removed: "CAN TERM FIT ONLY AT BUS END"
- board text removed: "GPS SMA"
- board text removed: "OIL"
- board text removed: "PI 5 VIDEO UART 3V3"
- board text removed: "RTC 3V NO CHARGE"
- board text removed: "SCREEN J10"
- board text removed: "TACH"
- board text removed: "THROTTLE"
